Commit message: add track simulation using simulink

File: src/simulation/ouster-gazebo-simulation/ouster_os1_64/urdf/os1_64.urdf.xacro (robot description, xacro)
@@ -3,5 +3,8 @@
 <robot xmlns:xacro="http://ros.org/wiki/xacro" name="os1_64">
   <xacro:property name="PI" value="3.1415926535897931"/>
-  <xacro:macro name="os1_64" params="*origin parent:=base name:=ouster reduced:=true prefix:=/os1_cloud_node hz:=10 samples:=512 min_range:=0.8 max_range:=100 noise:=0.008 min_angle_v:=-16.6 max_angle_v:=16.6 gpu:=false">
+  <xacro:macro name="os1_64" params="*origin parent:=base name:=ouster reduced:=true prefix:=/lidar hz:=10 samples:=512 min_range:=0.8 max_range:= 8 noise:=0.008 min_angle_v:=-16.6 max_angle_v:=16.6 gpu:=false">
+    <material name="Blue">
+      <color rgba="0.0 0.0 0.8 1.0"/>
+    </material>
     <!-- Conditional properties -->
     <xacro:if value="${reduced}">
@@ -40,4 +43,5 @@
           <mesh filename="package://ouster_os1_64/meshes/${file_visual}.stl" />
         </geometry>
+        <material name="Blue"/>
       </visual>
     </link>
@@ -50,56 +54,43 @@
     </joint>
     <gazebo reference="${name}_lidar">
-      <sensor type="${gpu_str}ray" name="${name}_lidar">
-        <pose>0 0 0 0 0 0</pose>
-        <visualize>false</visualize>
-        <update_rate>${hz}</update_rate>
-        <ray>
-          <scan>
-            <vertical>
-              <samples>64</samples>
-              <resolution>1</resolution>
-              <min_angle>${min_angle_v*PI/180.0}</min_angle>
-              <max_angle>${max_angle_v*PI/180.0}</max_angle>
-            </vertical>
-            <horizontal>
-              <samples>${samples}</samples>
-              <resolution>1</resolution>
-              <min_angle>-${PI}</min_angle>
-              <max_angle>${PI}</max_angle>
-            </horizontal>
-          </scan>
-          <range>
-            <min>${min_range}</min>
-            <max>${max_range}</max>
-            <resolution>0.03</resolution>
-          </range>
-          <noise>
-            <type>gaussian</type>
-            <mean>0.0</mean>
-            <stddev>0.000000000001</stddev>
-          </noise>
-        </ray>
-        <plugin name="gazebo_ros_laser_controller" filename="libgazebo_ros_ouster_${gpu_str}laser.so">
-          <topicName>${prefix}/points</topicName>
-          <frameName>${name}_lidar</frameName>
-          <min_range>${min_range}</min_range>
-          <max_range>${max_range}</max_range>
-          <gaussianNoise>${noise}</gaussianNoise>
-        </plugin>
-      </sensor>
-    </gazebo>
-    <link name="${name}_imu"/>
-    <joint name="${name}_imu_joint" type="fixed">
-      <parent link="${name}_sensor"/>
-      <child link="${name}_imu"/>
-    </joint>
-    <gazebo reference="${name}_imu">
-      <sensor type="imu" name="${name}_imu_sensor">
-        <pose>0 0 0 0 0 0</pose>
-        <always_on>true</always_on>
-        <update_rate>100</update_rate>
-        <visualize>true</visualize>
-        <topic>${prefix}/imu</topic>
-      </sensor>
+      <material>Gazebo/Blue </material>
+        <sensor type="${gpu_str}ray" name="${name}_lidar">
+          <pose>0 0 0 0 0 0</pose>
+          <visualize>false</visualize>
+          <update_rate>${hz}</update_rate>
+          <ray>
+            <scan>
+              <vertical>
+                <samples>64</samples>
+                <resolution>1</resolution>
+                <min_angle>${min_angle_v*PI/180.0}</min_angle>
+                <max_angle>${max_angle_v*PI/180.0}</max_angle>
+              </vertical>
+              <horizontal>
+                <samples>${samples}</samples>
+                <resolution>1</resolution>
+                <min_angle>-${PI*70/180}</min_angle>
+                <max_angle>${PI*70/180}</max_angle>
+              </horizontal>
+            </scan>
+            <range>
+              <min>${min_range}</min>
+              <max>${max_range}</max>
+              <resolution>0.03</resolution>
+            </range>
+            <noise>
+              <type>gaussian</type>
+              <mean>0.0</mean>
+              <stddev>0.000000000001</stddev>
+            </noise>
+          </ray>
+          <plugin name="gazebo_ros_laser_controller" filename="libgazebo_ros_ouster_${gpu_str}laser.so">
+            <topicName>${prefix}</topicName>
+            <frameName>${name}_lidar</frameName>
+            <min_range>${min_range}</min_range>
+            <max_range>${max_range}</max_range>
+            <gaussianNoise>${noise}</gaussianNoise>
+          </plugin>
+        </sensor>
     </gazebo>
   </xacro:macro>

File: src/simulation/ugv_sim/hunter/hunter2_base/urdf/hunter2_base_gazebo_os.xacro (robot description, xacro)
@@ -695,5 +695,5 @@
           <updateRate>0.0</updateRate>
           <cameraName>/camera_Right</cameraName>
-          <imageTopicName>image_raw</imageTopicName>
+          <imageTopicName>/usb_cam_right/image_raw</imageTopicName>
           <cameraInfoTopicName>camera_info</cameraInfoTopicName>
           <frameName>camera_link</frameName>
@@ -755,5 +755,5 @@
         <updateRate>0.0</updateRate>
         <cameraName>/camera_Left</cameraName>
-        <imageTopicName>image_raw</imageTopicName>
+        <imageTopicName>/usb_cam_left/image_raw</imageTopicName>
         <cameraInfoTopicName>camera_info</cameraInfoTopicName>
         <frameName>camera2_link</frameName>
